File: pcb/pcb.kicad_pcb (KiCad board)
At the start: 2 copper layers, 112 x 78 mm, 23 parts

Commit message: update
Parts:
- added ?: , Diode_SMD:D_SOD-323_HandSoldering, F.Cu at (21.9, 77.9)
- added ?: , Diode_SMD:D_SOD-323_HandSoldering, B.Cu at (21.9, 77.9)
- added ?: , Diode_SMD:D_SOD-323_HandSoldering, F.Cu at (39.9, 25.9)
- added ?: , Diode_SMD:D_SOD-323_HandSoldering, B.Cu at (39.9, 25.9)
- added ?: , Diode_SMD:D_SOD-323_HandSoldering, F.Cu at (39.9, 42.9)
- added ?: , Diode_SMD:D_SOD-323_HandSoldering, B.Cu at (39.9, 42.9)
- added ?: , Diode_SMD:D_SOD-323_HandSoldering, F.Cu at (21.9, 26.9)
- added ?: , Diode_SMD:D_SOD-323_HandSoldering, F.Cu at (39.9, 59.9)
- added ?: , Diode_SMD:D_SOD-323_HandSoldering, B.Cu at (39.9, 59.9)
- added ?: , Diode_SMD:D_SOD-323_HandSoldering, F.Cu at (39.9, 76.9)
- added ?: , Diode_SMD:D_SOD-323_HandSoldering, B.Cu at (39.9, 76.9)
- added ?: , Diode_SMD:D_SOD-323_HandSoldering, F.Cu at (57.9, 22.9)
- added ?: , Diode_SMD:D_SOD-323_HandSoldering, B.Cu at (57.9, 22.9)
- added ?: , Diode_SMD:D_SOD-323_HandSoldering, F.Cu at (57.9, 39.9)
- added ?: , Diode_SMD:D_SOD-323_HandSoldering, B.Cu at (21.9, 26.9)
- added ?: , Diode_SMD:D_SOD-323_HandSoldering, B.Cu at (57.9, 39.9)
- added ?: , Diode_SMD:D_SOD-323_HandSoldering, F.Cu at (57.9, 56.9)
- added ?: , Diode_SMD:D_SOD-323_HandSoldering, B.Cu at (57.9, 56.9)
- added ?: , Diode_SMD:D_SOD-323_HandSoldering, F.Cu at (57.9, 73.9)
- added ?: , Diode_SMD:D_SOD-323_HandSoldering, B.Cu at (57.9, 73.9)
- added ?: , Diode_SMD:D_SOD-323_HandSoldering, F.Cu at (75.9, 20.9)
- added ?: , Diode_SMD:D_SOD-323_HandSoldering, B.Cu at (75.9, 20.9)
- added ?: , Diode_SMD:D_SOD-323_HandSoldering, F.Cu at (75.9, 37.9)
- added ?: , Diode_SMD:D_SOD-323_HandSoldering, B.Cu at (75.9, 37.9)
- added ?: , Diode_SMD:D_SOD-323_HandSoldering, F.Cu at (75.9, 54.9)
- added ?: , Diode_SMD:D_SOD-323_HandSoldering, B.Cu at (75.9, 54.9)
- added ?: , Diode_SMD:D_SOD-323_HandSoldering, F.Cu at (75.9, 71.9)
- added ?: , Diode_SMD:D_SOD-323_HandSoldering, B.Cu at (75.9, 71.9)
- added ?: , Diode_SMD:D_SOD-323_HandSoldering, F.Cu at (21.9, 43.9)
- added ?: , Diode_SMD:D_SOD-323_HandSoldering, F.Cu at (93.9, 22.9)
- added ?: , Diode_SMD:D_SOD-323_HandSoldering, B.Cu at (93.9, 22.9)
- added ?: , Diode_SMD:D_SOD-323_HandSoldering, F.Cu at (93.9, 39.9)
- added ?: , Diode_SMD:D_SOD-323_HandSoldering, B.Cu at (93.9, 39.9)
- added ?: , Diode_SMD:D_SOD-323_HandSoldering, F.Cu at (93.9, 56.9)
- added ?: , Diode_SMD:D_SOD-323_HandSoldering, B.Cu at (93.9, 56.9)
- added ?: , Diode_SMD:D_SOD-323_HandSoldering, F.Cu at (93.9, 73.9)
- added ?: , Diode_SMD:D_SOD-323_HandSoldering, B.Cu at (21.9, 43.9)
- added ?: , Diode_SMD:D_SOD-323_HandSoldering, B.Cu at (93.9, 73.9)
- added ?: , Diode_SMD:D_SOD-323_HandSoldering, F.Cu at (111.9, 24.9)
- added ?: , Diode_SMD:D_SOD-323_HandSoldering, B.Cu at (111.9, 24.9)
- added ?: , Diode_SMD:D_SOD-323_HandSoldering, F.Cu at (111.9, 41.9)
- added ?: , Diode_SMD:D_SOD-323_HandSoldering, B.Cu at (111.9, 41.9)
- added ?: , Diode_SMD:D_SOD-323_HandSoldering, F.Cu at (111.9, 58.9)
- added ?: , Diode_SMD:D_SOD-323_HandSoldering, B.Cu at (111.9, 58.9)
- added ?: , Diode_SMD:D_SOD-323_HandSoldering, F.Cu at (21.9, 60.9)
- added ?: , Diode_SMD:D_SOD-323_HandSoldering, B.Cu at (21.9, 60.9)
Connections:
- ? pad 1: column_net -> (no net) (x23)
- ? pad 2: GND -> (no net) (x23)
Routing:
- net (no net): track 0.00 -> 1300.3 mm, vias 0 -> 46
